File: Xbox-Charge.kicad_sch (KiCad schematic)
At the start: 91 parts, among them J1 Conn_01x04_Pin, J2 Conn_01x04_Pin, Q1 CSD17551Q3A, Q2 CSD17551Q3A, Q3 CSD17551Q3A, Q4 CSD17551Q3A, Q5 CSD25402Q3A, U1 TPS25750, U2 BQ25713RSNR, U3 CAT24C512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

Commit message: Remove USB-C controller, planning to use MelonHD
Parts:
- removed C10, C11: 330pF, Capacitor_SMD:C_0201_0603Metric, symbol Device:C_Small
- removed C15, C16, C17: 10uF, Capacitor_SMD:C_0402_1005Metric, symbol Device:C_Small
- removed C18, C26: 0.1uF, Capacitor_SMD:C_0402_1005Metric, symbol Device:C_Small
- removed C19: 4.7uF, Capacitor_SMD:C_0805_2012Metric, symbol Device:C_Small
- removed C20, C21, C22, C23: 0.01uF, Capacitor_SMD:C_0402_1005Metric, symbol Device:C_Small
- removed C24, C25: 22uF, Capacitor_SMD:C_0805_2012Metric, symbol Device:C_Small
- removed C6, C7: 100uF, Capacitor_SMD:C_1210_3225Metric, symbol Device:C_Small
- removed C8, C9: 10uF, Capacitor_SMD:C_0603_1608Metric, symbol Device:C_Small
- removed JP1: Jumper_2_Open, Jumper:SolderJumper-2_P1.3mm_Open_RoundedPad1.0x1.5mm, symbol Jumper:Jumper_2_Open
- removed R3, R4, R5, R6, R7: 10K, Resistor_SMD:R_0402_1005Metric, symbol Device:R_Small
- removed U1: TPS25750, Xbox-Charge:TPS25750D, symbol TPS25750D:PTPS25750DRJKT
- removed U3: CAT24C512, Package_SO:SOIC-8_3.9x4.9mm_P1.27mm, symbol Memory_EEPROM:CAT24C512
- removed U4: TVS2200DRV, Package_SON:WSON-6-1EP_2x2mm_P0.65mm_EP1x1.6mm, symbol Power_Protection:TVS2200DRV
Other:
- moved on the sheet: BT1, C1, C12, C13, C14, C2, C27, C28, C29, C3, C30, C31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

Commit message: Rework 100W charge PCB, begin adding protection
Parts:
- removed C12, C13, C14, C27, C43, C44, C45, C46, C47, C5: 10uF, Capacitor_SMD:C_0805_2012Metric, symbol Device:C_Small
- removed J2: Conn_01x04_Pin, Xbox-Charge:VBUS PADS, symbol Connector:Conn_01x04_Pin
- added C5, C6: 100uF, Capacitor_Tantalum_SMD:CP_EIA-3216-18_Kemet-A, symbol Device:C_Polarized_Small
- added C7: 0.1uF, Capacitor_SMD:C_0402_1005Metric, symbol Device:C_Small
- added Q6, Q7, Q8, Q9: DMT3006, Package_DFN_QFN:Diodes_UDFN2020-6_Type-F, symbol Simulation_SPICE:NMOS
- added R3: 330, Resistor_SMD:R_0402_1005Metric, symbol Device:R_Small
- added R4: 2.2k, Resistor_SMD:R_0402_1005Metric, symbol Device:R_Small
- added R5, R6: 100k, Resistor_SMD:R_0402_1005Metric, symbol Device:R_Small
- added TP4: VBUS, TestPoint:TestPoint_Plated_Hole_D3.0mm, symbol Connector:TestPoint
- added TP5, TP7: GND, TestPoint:TestPoint_Plated_Hole_D3.0mm, symbol Connector:TestPoint
- added TP6: VSYS, TestPoint:TestPoint_Plated_Hole_D3.0mm, symbol Connector:TestPoint
- added U1: BQ297xy, Package_SON:WSON-6_1.5x1.5mm_P0.5mm, symbol Battery_Management:BQ297xy
Connections:
- net GND: now also C5.2, C6.2, Q8.1 (D), Q8.2 (D), Q8.5 (D), Q8.6 (D), Q8.7 (D), Q9.4 (S), Q9.8 (S), R6.2, TP5.1, TP7.1; no longer BT1.2 (-), TP3.1
- net VBUS: now also C6.1, TP4.1
- net BATT+: now reaches BT1.1 (+), C28.1, R10.2, R12.1, TP2.1
- net BATT+: now also R3.2
- net VSYS renamed VCC
- net VCC: now also C5.1, R5.2, TP6.1
- new net: R4.2, U1.6 (V-)
- new net: Q6.1 (D), Q6.2 (D), Q6.5 (D), Q6.6 (D), Q6.7 (D), Q7.1 (D), Q7.2 (D), Q7.5 (D), Q7.6 (D), Q7.7 (D)
- new net: Q6.3 (G), U1.3 (Dout)
- new net: Q8.3 (G), Q9.1 (D), Q9.2 (D), Q9.5 (D), Q9.6 (D), Q9.7 (D), R5.1
- new net: C7.1, R3.1, U1.5 (BAT)
- new net: Q7.3 (G), U1.2 (Cout)
- new net BATT-: BT1.2 (-), C7.2, Q6.4 (S), Q6.8 (S), TP3.1, U1.4 (VSS)
- new net BATT-_2: Q7.4 (S), Q7.8 (S), Q8.4 (S), Q8.8 (S), R4.1
- new net SHIP: Q9.3 (G), R6.1
Other:
- moved on the sheet: BT1, C42, TP2, TP3

Commit message: misc improvements
Parts:
- removed Q9: DMT3006, Package_DFN_QFN:Diodes_UDFN2020-6_Type-F, symbol Simulation_SPICE:NMOS
- removed R6: 100k, Resistor_SMD:R_0402_1005Metric, symbol Device:R_Small
- added C8, C9: 100uF, Capacitor_Tantalum_SMD:CP_EIA-3216-18_Kemet-A, symbol Device:C_Polarized_Small
- added D1: BAT54C, Package_TO_SOT_SMD:SOT-23-3, symbol Diode:BAT54C
- added R7: 100k, Resistor_SMD:R_0402_1005Metric, symbol Device:R_Small
- added TP8: ~{SHIP}, TestPoint:TestPoint_Pad_D1.5mm, symbol Connector:TestPoint
- U1: Digikey (none) -> https://www.digikey.com.au/en/products/detail/texas-instrum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
Connections:
- net GND: now also C8.2, C9.2
- net VBUS: now also C9.1, R7.2
- net VCC: now also C8.1
- net at R5.1: now also D1.1; no longer Q8.3 (G)
- new net: D1.2, R7.1
- new net ~{SHIP}: D1.3, Q8.3 (G), TP8.1
Other:
- moved on the sheet: BT1, C7, Q6, Q7, Q8, R3, R4, R5, TP2, TP3, U1
